File: examples/spice-parser/kicad-pyspice-example/kicad-pyspice-example.sch (KiCad schematic (older format))
At the start: 7 parts, among them X1 JackIn, X2 PowerIn, X3 Opamp, X4 JackOut

Commit message: refactor: changint the name from PySpice to InSpice
Parts:
- R1, R2, R3: symbol R-RESCUE-kicad-pyspice-example -> R-RESCUE-kicad-InSpice-example
- X3: symbol LM193-RESCUE-kicad-pyspice-example -> LM193-RESCUE-kicad-InSpice-example
Changed lines of the file:
@@
 EESchema Schematic File Version 2
-LIBS:kicad-pyspice-example-rescue
+LIBS:kicad-InSpice-example-rescue
 LIBS:power
 LIBS:device
@@
 LIBS:memory
 LIBS:xilinx
-LIBS:kicad-pyspice-example-cache
+LIBS:kicad-InSpice-example-cache
 EELAYER 25 0
 EELAYER END
@@
 $EndDescr
 $Comp
-L LM193-RESCUE-kicad-pyspice-example X3
+L LM193-RESCUE-kicad-InSpice-example X3
 U 1 1 55381082
 P 5450 3750
@@
 $EndComp
 $Comp
-L R-RESCUE-kicad-pyspice-example R2
+L R-RESCUE-kicad-InSpice-example R2
 U 1 1 553812CC
 P 5850 4200
@@
 $EndComp
 $Comp
-L R-RESCUE-kicad-pyspice-example R1
+L R-RESCUE-kicad-InSpice-example R1
 U 1 1 553812DB
 P 4450 3850
@@
 $EndComp
 $Comp
-L GND-RESCUE-kicad-pyspice-example #PWR01
+L GND-RESCUE-kicad-InSpice-example #PWR01
 U 1 1 553813CF
 P 4750 4900
@@
 $EndComp
 $Comp
-L GND-RESCUE-kicad-pyspice-example #PWR04
+L GND-RESCUE-kicad-InSpice-example #PWR04
 U 1 1 55381612
 P 4450 3150
@@
 	6750 4000 6750 4750
 $Comp
-L R-RESCUE-kicad-pyspice-example R3
+L R-RESCUE-kicad-InSpice-example R3
 U 1 1 5538F1ED
 P 6550 4300
